Commit message: Starting simulation package

File: two_wheel_urdf/urdf/two_wheel.xacro (robot description, xacro)
@@ -1,4 +1,6 @@
 <?xml version="1.0"?>
 <robot name="two_wheel" xmlns:xacro="http://ros.org/wiki/xacro">
+<!-- Constants for robot dimensions -->
+  <xacro:property name="base_link_size" value="0.5 0.5 0.25" />
   <!-- Base Link -->
   <link name="base_link">
@@ -6,5 +8,5 @@
       <origin xyz="0 0 0" rpy="0 0 0" />
       <geometry>
-          <box size="0.5 0.5 0.25"/>
+          <box size="${base_link_size}"/>
       </geometry>
       <material name="white">
@@ -16,5 +18,5 @@
       <origin xyz="0 0 0" rpy="0 0 0" />
       <geometry>
-          <box size="0.5 0.5 0.25"/>
+          <box size="${base_link_size}"/>
       </geometry>
     </collision>
