Commit message: Adding update

File: two_wheel_simulation/urdf/two_wheel.xacro (robot description, xacro)
@@ -24,5 +24,5 @@
     <!-- Caster -->
     <visual name="caster">
-      <origin xyz="0.2 0 -0.125" rpy="0 0 0" />
+      <origin xyz="-0.2 0 -0.125" rpy="0 0 0" />
       <geometry>
         <sphere radius="0.05" />
@@ -31,5 +31,5 @@
     <!-- Caster collision, mass and inertia -->
     <collision>
-      <origin xyz="0.2 0 -0.125" rpy="0 0 0" />
+      <origin xyz="-0.2 0 -0.125" rpy="0 0 0" />
       <geometry>
         <sphere radius="0.05" />
